File: PCB-2-3inch-7seg-HEF4094B/PCB-2-3inch-7seg-HEF4094B.sch (KiCad schematic (older format))
At the start: 26 parts

Commit message: finalize sch
Parts:
- removed R? (x14): 470, symbol Device:R_Small
- added C5, C6: 0.1u, Capacitor_SMD:C_0805_2012Metric, symbol Device:C_Small
- added D1: D_Small, Diode_SMD:D_SMA, symbol Device:D_Small
- added H1, H2, H3, H4: mount, MountingHole:MountingHole_3.5mm_Pad, symbol Mechanical:MountingHole_Pad
- added J1: IN, Connector_PinSocket_2.54mm:PinSocket_1x05_P2.54mm_Vertical, symbol Connector_Generic:Conn_01x05
- added J2: OUT, Connector_PinSocket_2.54mm:PinSocket_1x05_P2.54mm_Vertical, symbol Connector_Generic:Conn_01x05
- added R10, R11, R12, R13, R14, R15, R16, R3, R4, R5, R6, R7, R8, R9: 470, Resistor_SMD:R_0805_2012Metric_Pad1.15x1.40mm_HandSolder, symbol Device:R_Small
- added U7: KA78M05_TO252, Package_TO_SOT_SMD:TO-252-2, symbol Regulator_Linear:KA78M05_TO252
- C1, C2, C3, C4: renamed from C?; footprint (none) -> Capacitor_SMD:C_0805_2012Metric
- R1, R2: renamed from R?; footprint (none) -> Resistor_SMD:R_0805_2012Metric_Pad1.15x1.40mm_HandSolder
- U1, U2: renamed from U?; footprint SOIC127P600X175-16N -> Package_SO:SOIC-16_3.9x9.9mm_P1.27mm
- U4: renamed from U?; footprint (none) -> Package_SO:SOP-18_7x12.5mm_P1.27mm
- U5, U6: renamed from U?; value SA15-11SRWA -> 23011; footprint Display_7Segment:SA15-11xxx -> Display_7Segment:23011-7-segment
- gave numbers to parts that had none: 1
Connections:
- net +12V: now also D1.2 (A), J1.1 (Pin_1), J2.1 (Pin_1)
- net +5V: now also C6.1, U7.3 (VO)
- net CLK: now also J1.3 (Pin_3), J2.3 (Pin_3)
- net DIN0: now also J1.5 (Pin_5)
- net DOUT1: now also J2.5 (Pin_5)
- net GND: now also C5.2, C6.2, J1.2 (Pin_2), J2.2 (Pin_2), U7.2 (GND)
- net STR: now also J1.4 (Pin_4), J2.4 (Pin_4)
- net at U3.11 (O8): now also R8.2
- net at U3.12 (O7): now also R7.2
- net at U3.13 (O6): now also R6.2
- net at U3.14 (O5): now also R5.2
- net at U3.15 (O4): now also R4.2
- net at U3.16 (O3): now also R3.2
- net at U5.10 (G): now also R7.1
- net at U5.2 (E): now also R5.1
- net at U5.3 (D): now also R4.1
- net at U5.4 (C): now also R3.1
- net at U5.8 (DP): now also R8.1
- net at U5.9 (F): now also R6.1
- net at U4.11 (O8): now also R16.2
- net at U4.12 (O7): now also R15.2
- net at U4.13 (O6): now also R14.2
- net at U4.14 (O5): now also R13.2
- net at U4.15 (O4): now also R12.2
- net at U4.16 (O3): now also R11.2
- net at U4.17 (O2): now also R10.2
- net at U4.18 (O1): now also R9.2
- net at U6.10 (G): now also R15.1
- net at U6.2 (E): now also R13.1
- net at U6.3 (D): now also R12.1
- net at U6.4 (C): now also R11.1
- net at U6.6 (B): now also R10.1
- net at U6.7 (A): now also R9.1
- net at U6.8 (DP): now also R16.1
- net at U6.9 (F): now also R14.1
- new net: C5.1, D1.1 (K), U7.1 (VI)

Commit message: finalize pcb v1.0
Parts:
- R1, R10, R11, R12, R13, R14, R15, R16, R2, R3, R4, R5, R6, R7, R8, R9: footprint Resistor_SMD:R_0805_2012Metric_Pad1.15x1.40mm_HandSolder -> Resistor_THT:R_Axial_DIN0207_L6.3mm_D2.5mm_P10.16mm_Horizontal
Changed lines of the file:
@@
 F 0 "R1" V 8200 2200 50  0000 C CNN
 F 1 "470" V 8200 2475 50  0000 C CNN
-F 2 "Resistor_SMD:R_0805_2012Metric_Pad1.15x1.40mm_HandSolder" H 8250 2325 50  0001 C CNN
+F 2 "Resistor_THT:R_Axial_DIN0207_L6.3mm_D2.5mm_P10.16mm_Horizontal" H 8250 2325 50  0001 C CNN
 F 3 "~" H 8250 2325 50  0001 C CNN
 	1    8250 2325
@@
 Wire Wire Line
 	8350 2325 8575 2325
-$Comp
-L Device:R_Small R2
-U 1 1 5F2B51F9
-P 8250 2425
-F 0 "R2" V 8200 2300 50  0000 C CNN
-F 1 "470" V 8200 2575 50  0000 C CNN
-F 2 "Resistor_SMD:R_0805_2012Metric_Pad1.15x1.40mm_HandSolder" H 8250 2425 50  0001 C CNN
-F 3 "~" H 8250 2425 50  0001 C CNN
-	1    8250 2425
-	0    1    1    0
-$EndComp
 Wire Wire Line
 	8150 2425 7875 2425
@@
 Connection ~ 3375 5650
 $Comp
+L Device:R_Small R2
+U 1 1 5F3392C6
+P 8250 2425
+F 0 "R2" V 8200 2300 50  0000 C CNN
+F 1 "470" V 8200 2575 50  0000 C CNN
+F 2 "Resistor_THT:R_Axial_DIN0207_L6.3mm_D2.5mm_P10.16mm_Horizontal" H 8250 2425 50  0001 C CNN
+F 3 "~" H 8250 2425 50  0001 C CNN
+	1    8250 2425
+	0    1    1    0
+$EndComp
+$Comp
 L Device:R_Small R3
-U 1 1 5F3C09A1
+U 1 1 5F33DF74
 P 8250 2525
 F 0 "R3" V 8200 2400 50  0000 C CNN
 F 1 "470" V 8200 2675 50  0000 C CNN
-F 2 "Resistor_SMD:R_0805_2012Metric_Pad1.15x1.40mm_HandSolder" H 8250 2525 50  0001 C CNN
+F 2 "Resistor_THT:R_Axial_DIN0207_L6.3mm_D2.5mm_P10.16mm_Horizontal" H 8250 2525 50  0001 C CNN
 F 3 "~" H 8250 2525 50  0001 C CNN
 	1    8250 2525
@@
 $Comp
 L Device:R_Small R4
-U 1 1 5F3C5697
+U 1 1 5F342B70
 P 8250 2625
 F 0 "R4" V 8200 2500 50  0000 C CNN
 F 1 "470" V 8200 2775 50  0000 C CNN
-F 2 "Resistor_SMD:R_0805_2012Metric_Pad1.15x1.40mm_HandSolder" H 8250 2625 50  0001 C CNN
+F 2 "Resistor_THT:R_Axial_DIN0207_L6.3mm_D2.5mm_P10.16mm_Horizontal" H 8250 2625 50  0001 C CNN
 F 3 "~" H 8250 2625 50  0001 C CNN
 	1    8250 2625
@@
 $Comp
 L Device:R_Small R5
-U 1 1 5F3CA273
+U 1 1 5F3476F9
 P 8250 2725
 F 0 "R5" V 8200 2600 50  0000 C CNN
 F 1 "470" V 8200 2875 50  0000 C CNN
-F 2 "Resistor_SMD:R_0805_2012Metric_Pad1.15x1.40mm_HandSolder" H 8250 2725 50  0001 C CNN
+F 2 "Resistor_THT:R_Axial_DIN0207_L6.3mm_D2.5mm_P10.16mm_Horizontal" H 8250 2725 50  0001 C CNN
 F 3 "~" H 8250 2725 50  0001 C CNN
 	1    8250 2725
@@
 $Comp
 L Device:R_Small R6
-U 1 1 5F3CEEA8
+U 1 1 5F34C2AC
 P 8250 2825
 F 0 "R6" V 8200 2700 50  0000 C CNN
 F 1 "470" V 8200 2975 50  0000 C CNN
-F 2 "Resistor_SMD:R_0805_2012Metric_Pad1.15x1.40mm_HandSolder" H 8250 2825 50  0001 C CNN
+F 2 "Resistor_THT:R_Axial_DIN0207_L6.3mm_D2.5mm_P10.16mm_Horizontal" H 8250 2825 50  0001 C CNN
 F 3 "~" H 8250 2825 50  0001 C CNN
 	1    8250 2825
@@
 $Comp
 L Device:R_Small R7
-U 1 1 5F3D3A8F
+U 1 1 5F350EE7
 P 8250 2925
 F 0 "R7" V 8200 2800 50  0000 C CNN
 F 1 "470" V 8200 3075 50  0000 C CNN
-F 2 "Resistor_SMD:R_0805_2012Metric_Pad1.15x1.40mm_HandSolder" H 8250 2925 50  0001 C CNN
+F 2 "Resistor_THT:R_Axial_DIN0207_L6.3mm_D2.5mm_P10.16mm_Horizontal" H 8250 2925 50  0001 C CNN
 F 3 "~" H 8250 2925 50  0001 C CNN
 	1    8250 2925
@@
 $Comp
 L Device:R_Small R8
-U 1 1 5F3D86F4
+U 1 1 5F355B70
 P 8250 3025
 F 0 "R8" V 8200 2900 50  0000 C CNN
 F 1 "470" V 8200 3175 50  0000 C CNN
-F 2 "Resistor_SMD:R_0805_2012Metric_Pad1.15x1.40mm_HandSolder" H 8250 3025 50  0001 C CNN
+F 2 "Resistor_THT:R_Axial_DIN0207_L6.3mm_D2.5mm_P10.16mm_Horizontal" H 8250 3025 50  0001 C CNN
 F 3 "~" H 8250 3025 50  0001 C CNN
 	1    8250 3025
@@
 $Comp
 L Device:R_Small R9
-U 1 1 5F3DD3DF
+U 1 1 5F35F3A1
 P 8250 4325
 F 0 "R9" V 8200 4200 50  0000 C CNN
 F 1 "470" V 8200 4475 50  0000 C CNN
-F 2 "Resistor_SMD:R_0805_2012Metric_Pad1.15x1.40mm_HandSolder" H 8250 4325 50  0001 C CNN
+F 2 "Resistor_THT:R_Axial_DIN0207_L6.3mm_D2.5mm_P10.16mm_Horizontal" H 8250 4325 50  0001 C CNN
 F 3 "~" H 8250 4325 50  0001 C CNN
 	1    8250 4325
@@
 $Comp
 L Device:R_Small R10
-U 1 1 5F3E70C2
+U 1 1 5F363F8D
 P 8250 4425
 F 0 "R10" V 8200 4300 50  0000 C CNN
 F 1 "470" V 8200 4575 50  0000 C CNN
-F 2 "Resistor_SMD:R_0805_2012Metric_Pad1.15x1.40mm_HandSolder" H 8250 4425 50  0001 C CNN
+F 2 "Resistor_THT:R_Axial_DIN0207_L6.3mm_D2.5mm_P10.16mm_Horizontal" H 8250 4425 50  0001 C CNN
 F 3 "~" H 8250 4425 50  0001 C CNN
 	1    8250 4425
@@
 $Comp
 L Device:R_Small R11
-U 1 1 5F3EBE00
+U 1 1 5F368B74
 P 8250 4525
 F 0 "R11" V 8200 4400 50  0000 C CNN
 F 1 "470" V 8200 4675 50  0000 C CNN
-F 2 "Resistor_SMD:R_0805_2012Metric_Pad1.15x1.40mm_HandSolder" H 8250 4525 50  0001 C CNN
+F 2 "Resistor_THT:R_Axial_DIN0207_L6.3mm_D2.5mm_P10.16mm_Horizontal" H 8250 4525 50  0001 C CNN
 F 3 "~" H 8250 4525 50  0001 C CNN
 	1    8250 4525
@@
 $Comp
 L Device:R_Small R12
-U 1 1 5F3F0A54
+U 1 1 5F36D6D3
 P 8250 4625
 F 0 "R12" V 8200 4500 50  0000 C CNN
 F 1 "470" V 8200 4775 50  0000 C CNN
-F 2 "Resistor_SMD:R_0805_2012Metric_Pad1.15x1.40mm_HandSolder" H 8250 4625 50  0001 C CNN
+F 2 "Resistor_THT:R_Axial_DIN0207_L6.3mm_D2.5mm_P10.16mm_Horizontal" H 8250 4625 50  0001 C CNN
 F 3 "~" H 8250 4625 50  0001 C CNN
 	1    8250 4625
@@
 $Comp
 L Device:R_Small R13
-U 1 1 5F3F568C
+U 1 1 5F3723AC
 P 8250 4725
 F 0 "R13" V 8200 4600 50  0000 C CNN
 F 1 "470" V 8200 4875 50  0000 C CNN
-F 2 "Resistor_SMD:R_0805_2012Metric_Pad1.15x1.40mm_HandSolder" H 8250 4725 50  0001 C CNN
+F 2 "Resistor_THT:R_Axial_DIN0207_L6.3mm_D2.5mm_P10.16mm_Horizontal" H 8250 4725 50  0001 C CNN
 F 3 "~" H 8250 4725 50  0001 C CNN
 	1    8250 4725
@@
 $Comp
 L Device:R_Small R14
-U 1 1 5F3FA446
+U 1 1 5F376FC8
 P 8250 4825
 F 0 "R14" V 8200 4700 50  0000 C CNN
 F 1 "470" V 8200 4975 50  0000 C CNN
-F 2 "Resistor_SMD:R_0805_2012Metric_Pad1.15x1.40mm_HandSolder" H 8250 4825 50  0001 C CNN
+F 2 "Resistor_THT:R_Axial_DIN0207_L6.3mm_D2.5mm_P10.16mm_Horizontal" H 8250 4825 50  0001 C CNN
 F 3 "~" H 8250 4825 50  0001 C CNN
 	1    8250 4825
@@
 $Comp
 L Device:R_Small R15
-U 1 1 5F3FF003
+U 1 1 5F37BBE9
 P 8250 4925
 F 0 "R15" V 8200 4800 50  0000 C CNN
 F 1 "470" V 8200 5075 50  0000 C CNN
-F 2 "Resistor_SMD:R_0805_2012Metric_Pad1.15x1.40mm_HandSolder" H 8250 4925 50  0001 C CNN
+F 2 "Resistor_THT:R_Axial_DIN0207_L6.3mm_D2.5mm_P10.16mm_Horizontal" H 8250 4925 50  0001 C CNN
 F 3 "~" H 8250 4925 50  0001 C CNN
 	1    8250 4925
@@
 $Comp
 L Device:R_Small R16
-U 1 1 5F403D0A
+U 1 1 5F3807E5
 P 8250 5025
 F 0 "R16" V 8200 4900 50  0000 C CNN
 F 1 "470" V 8200 5175 50  0000 C CNN
-F 2 "Resistor_SMD:R_0805_2012Metric_Pad1.15x1.40mm_HandSolder" H 8250 5025 50  0001 C CNN
+F 2 "Resistor_THT:R_Axial_DIN0207_L6.3mm_D2.5mm_P10.16mm_Horizontal" H 8250 5025 50  0001 C CNN
 F 3 "~" H 8250 5025 50  0001 C CNN
 	1    8250 5025
