File: PCB-2-3inch-7seg-HEF4094B/PCB-2-3inch-7seg-HEF4094B.kicad_pcb (KiCad board)
At the start: 2 copper layers, 72.9 x 88.1 mm, 36 parts, among them J1 IN, J2 OUT, U1 HEF4094BT,653, U2 HEF4094BT,653, U3 ULN2803A, U4 ULN2803A, U5 23011, U6 23011, U7 KA78M05_TO252

Commit message: finalize pcb v1.0
Parts:
- R1, R10, R11, R12, R13, R14, R15, R16, R2, R3, R4, R5, R6, R7, R8, R9: footprint Resistor_SMD:R_0805_2012Metric_Pad1.15x1.40mm_HandSolder -> Resistor_THT:R_Axial_DIN0207_L6.3mm_D2.5mm_P10.16mm_Horizontal; moved to F.Cu
- moved C5 158.3 mm to (135.6, 49.1), turned to 180 degrees
- moved C6 135.2 mm to (151.2, 87.9), turned to 270 degrees
- moved C2 131.8 mm to (124.7, 87.4), turned to 270 degrees
- moved C3 130.6 mm to (149.4, 52.1), turned to 180 degrees
- moved D1 130.5 mm to (142.9, 49.1)
- moved C1 126.5 mm to (140.0, 59.8), turned to 180 degrees
- moved C4 123.7 mm to (149.4, 49.1), turned to 180 degrees
- moved R11 83.6 mm to (162.1, 103.1), turned to 90 degrees
- moved R5 80.7 mm to (129.7, 103.3), turned to 90 degrees
- moved R13 78.3 mm to (156.0, 103.1), turned to 90 degrees
- moved R12 77.9 mm to (159.0, 103.1), turned to 90 degrees
- moved R4 77.6 mm to (132.7, 103.3), turned to 90 degrees
- moved R3 76.6 mm to (135.7, 103.3), turned to 90 degrees
- moved U7 67.4 mm to (136.7, 54.8), turned to 180 degrees
- moved R6 48.8 mm to (113.5, 55.4), turned to 270 degrees
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Routing:
- net GND: track 0.00 -> 421.7 mm, vias 0 -> 2
- net +12V: track 133.1 -> 291.6 mm, vias 0 -> 2
- net +5V: track 1.27 -> 148.0 mm, vias 0 -> 2
- net /CLK: track 10.0 -> 148.9 mm, vias 2 -> 0
- net /STR: track 14.5 -> 117.3 mm
- net /DOUT1: track 0.00 -> 65.9 mm, vias 0 -> 2
- net /DOUT0: track 0.00 -> 63.3 mm, vias 0 -> 2
- net Net-(U2-Pad4): track 15.7 -> 47.0 mm
- net Net-(U1-Pad4): track 16.8 -> 43.0 mm
- net Net-(U2-Pad5): track 16.7 -> 41.7 mm
- net Net-(R3-Pad1): track 0.00 -> 22.3 mm
- net Net-(R4-Pad1): track 0.00 -> 21.5 mm
- net Net-(R4-Pad2): track 33.0 -> 12.7 mm
- net Net-(R5-Pad1): track 0.00 -> 20.2 mm
- net Net-(R5-Pad2): track 35.6 -> 15.4 mm
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
Commit message: DIY print
Parts:
- added G***: LOGO, Symbol:T_logo, B.Cu at (140.3, 41.0)
Routing:
- net +5V: track 148.0 -> 150.0 mm
- net GND: track 421.7 -> 422.7 mm
- net Net-(U1-Pad4): track 43.0 -> 43.9 mm
- net Net-(R13-Pad2): track 15.4 -> 16.3 mm
- net Net-(U1-Pad5): track 37.4 -> 38.2 mm
- net Net-(U1-Pad6): track 31.9 -> 32.6 mm
- net Net-(R12-Pad2): track 12.9 -> 13.5 mm
- net Net-(R5-Pad2): track 15.4 -> 16.0 mm
- net Net-(R1-Pad2): track 42.0 -> 42.6 mm
- net Net-(R6-Pad2): track 47.6 -> 48.1 mm
- net Net-(U1-Pad7): track 26.5 -> 27.1 mm
- net Net-(R14-Pad2): track 25.6 -> 26.1 mm
- net Net-(U2-Pad4): track 47.0 -> 47.5 mm
Other:
- board text added: "theara - 093 568 593"
